Commit message: modify new LeapHandFlip env from LeapHandRot

File: leap_sim/assets/leap_hand/leaphand_cube.urdf (robot description, URDF)
Before this commit: robot leap_hand, 27 links, 26 joints
Links:
- link palm_lower: geometry collision box size=0.035 0.115 0.025; collision box size=0.04 0.063 0.025
Joints:
- joint world2hand: origin xyz=0 0 0.5 rpy=3.14159265 0 0 -> xyz=0 0 0 rpy=3.14159265 0 0
