Commit message: update for taskB (#16)
* modified LeapHandFlip env

* add LfD method for LeapHandFlip, not working at all

* 1) separate fingertip rigid/soft part in CAD, 2) add rigid-penalty & soft-reward for fingertip contact, 3) lower ftip_cf_scale for LeapHandFlip env

* raise palm height and object init height for LeapHandFlip env

* add dof effort limit to LeapHandFlip and LeapHandRot envs

* add reset_object strategy to center the object before deploying RL

* add action_lib to connect agent_hw&taskB_highlevel

* add doc for taskB

File: leap_sim/assets/leap_hand/leaphand_high_palm.urdf (robot description, URDF)
Before this commit: robot leap_hand, 26 links, 25 joints
Links:
- removed link fingertip_2_new
- removed link fingertip_3_new
- removed link fingertip_new
- removed link thumb_fingertip_new
- added link fingertip_2_new_root, mass 0.005; collision mesh filename=fingertip_custom_root.stl; visual mesh filename=fingertip_custom.stl
- added link fingertip_2_new_tip, mass 0.01; collision mesh filename=fingertip_custom_tip.stl
- added link fingertip_3_new_root, mass 0.005; collision mesh filename=fingertip_custom_root.stl; visual mesh filename=fingertip_custom.stl
- added link fingertip_3_new_tip, mass 0.01; collision mesh filename=fingertip_custom_tip.stl
- added link fingertip_new_root, mass 0.005; collision mesh filename=fingertip_custom_root.stl; visual mesh filename=fingertip_custom.stl
- added link fingertip_new_tip, mass 0.01; collision mesh filename=fingertip_custom_tip.stl
- added link thumb_fingertip_new_root, mass 0.005; collision mesh filename=fingertip_custom_root.stl; visual mesh filename=fingertip_custom.stl
- added link thumb_fingertip_new_tip, mass 0.01; collision mesh filename=fingertip_custom_tip.stl
Joints:
- removed joint finger1_tipbase2tip
- removed joint finger2_tipbase2tip
- removed joint finger3_tipbase2tip
- removed joint thumb_tipbase2tip
- added joint finger1_tipbase2root: type fixed, parent fingertip, child fingertip_new_root, origin xyz=0 -0.017 0.0145 rpy=0 1.5707963267948966 3.141592653589793
- added joint finger1_tiproot2tip: type fixed, parent fingertip_new_root, child fingertip_new_tip, origin xyz=0 0 0 rpy=0 0 0
- added joint finger2_tipbase2root: type fixed, parent fingertip_2, child fingertip_2_new_root, origin xyz=0 -0.017 0.0145 rpy=0 1.5707963267948966 3.141592653589793
- added joint finger2_tiproot2tip: type fixed, parent fingertip_2_new_root, child fingertip_2_new_tip, origin xyz=0 0 0 rpy=0 0 0
- added joint finger3_tipbase2root: type fixed, parent fingertip_3, child fingertip_3_new_root, origin xyz=0 -0.017 0.0145 rpy=0 1.5707963267948966 3.141592653589793
- added joint finger3_tiproot2tip: type fixed, parent fingertip_3_new_root, child fingertip_3_new_tip, origin xyz=0 0 0 rpy=0 0 0
- added joint thumb_tipbase2root: type fixed, parent thumb_fingertip, child thumb_fingertip_new_root, origin xyz=0 -0.03 -0.0145 rpy=0 1.5707963267948966 3.141592653589793
- added joint thumb_tiproot2tip: type fixed, parent thumb_fingertip_new_root, child thumb_fingertip_new_tip, origin xyz=0 0 0 rpy=0 0 0
- joint finger1_tip2center: parent fingertip_new -> fingertip_new_tip
- joint finger2_tip2center: parent fingertip_2_new -> fingertip_2_new_tip
- joint finger3_tip2center: parent fingertip_3_new -> fingertip_3_new_tip
- joint thumb_tip2center: parent thumb_fingertip_new -> thumb_fingertip_new_tip
