Commit message: add code for RA-P experiments

File: my_robot_description/urdf/leap_hand/leap_hand_body.urdf.xacro (robot description, xacro)
@@ -177,4 +177,5 @@
             <limit effort="0.95" velocity="8.48" lower="-1.047" upper="1.047" />
             <joint_properties friction="0.0" />
+            <dynamics D="1" K="7000" damping="0.003" friction="0.0" mu_coulomb="0" mu_viscous="16" />
         </joint>
         <joint name="joint_1" type="revolute">

File: my_robot_description/urdf/leaphand.urdf.xacro (robot description, xacro)
@@ -1,15 +1,17 @@
 <?xml version="1.0"?>
 <robot name="leap_hand" xmlns:xacro="http://www.ros.org/wiki/xacro">
-	<!-- using ros -->
-	<!-- <xacro:arg name="package_dir" default="package://my_robot_description" /> -->
-	<!-- using absolute path (for generating urdf)-->
-	<!-- <xacro:arg name="package_dir" default="/home/mingrui/Mingrui/research/project_RGMC_24/RGMC_XL/leap_ws/src/my_robot_description" /> -->
+    <!-- using ros -->
+    <!-- <xacro:arg name="package_dir" default="package://my_robot_description" /> -->
+    <!-- using absolute path (for generating urdf)-->
+    <!-- <xacro:arg name="package_dir" default="/home/mingrui/Mingrui/research/project_RGMC_24/RGMC_XL/leap_ws/src/my_robot_description" /> -->
     <!-- <xacro:arg name="mesh_dir" default="$(arg package_dir)/urdf/leap_hand/mesh/" /> -->
     <!-- specify the mesh_dir -->
     <!-- <xacro:arg name="mesh_dir" default="" /> -->
     <xacro:arg name="mesh_dir" default="package://my_robot_description/urdf/leap_hand/mesh/" />
-    <!-- <xacro:arg name="mesh_dir" default="/home/mingrui/Mingrui/research/project_RGMC_24/RGMC_XL/leap_ws/src/my_robot_description/urdf/leap_hand/mesh/" /> -->
-	<xacro:include filename="$(find my_robot_description)/urdf/leap_hand/leap_hand_body.urdf.xacro"/>
-    <xacro:leap_hand_body mesh_dir="$(arg mesh_dir)"/>
+    <!-- <xacro:arg name="mesh_dir"
+    default="/home/mingrui/Mingrui/research/project_RGMC_24/RGMC_XL/leap_ws/src/my_robot_description/urdf/leap_hand/mesh/" /> -->
+    <!-- <xacro:arg name="mesh_dir" default="package://drake_models/leap_description/meshes/" /> -->
+    <xacro:include filename="$(find my_robot_description)/urdf/leap_hand/leap_hand_body.urdf.xacro" />
+    <xacro:leap_hand_body mesh_dir="$(arg mesh_dir)" />
     <!-- the links and joints for customized fingertips -->
     <link name="fingertip_new">
@@ -17,8 +19,8 @@
             <origin xyz="0 0 0" rpy="0 0 0" />
             <geometry>
-            <mesh filename="$(arg mesh_dir)fingertip_custom.stl"/>
+                <mesh filename="$(arg mesh_dir)fingertip_custom.stl" />
             </geometry>
             <material name="fingertip_material">
-            <color rgba="0.86666666666666669627 0.86666666666666669627 0.050980392156862744391 1.0"/>
+                <color rgba="0.86666666666666669627 0.86666666666666669627 0.050980392156862744391 1.0" />
             </material>
         </visual>
@@ -26,11 +28,11 @@
             <origin xyz="0 0 0" rpy="0 0 0" />
             <geometry>
-            <mesh filename="$(arg mesh_dir)fingertip_custom.stl"/>
+                <mesh filename="$(arg mesh_dir)fingertip_custom.stl" />
             </geometry>
         </collision>
         <inertial>
-            <origin xyz="0 0 0" rpy="0 0 0"/>
+            <origin xyz="0 0 0" rpy="0 0 0" />
             <mass value="0.0000000001" />
-            <inertia ixx="0.0000000001" ixy="0"  ixz="0" iyy="0.0000000001" iyz="0" izz="0.0000000001" />
+            <inertia ixx="0.0000000001" ixy="0" ixz="0" iyy="0.0000000001" iyz="0" izz="0.0000000001" />
         </inertial>
     </link>
@@ -39,8 +41,8 @@
             <origin xyz="0 0 0" rpy="0 0 0" />
             <geometry>
-            <mesh filename="$(arg mesh_dir)fingertip_custom.stl"/>
+                <mesh filename="$(arg mesh_dir)fingertip_custom.stl" />
             </geometry>
             <material name="fingertip_material">
-            <color rgba="0.86666666666666669627 0.86666666666666669627 0.050980392156862744391 1.0"/>
+                <color rgba="0.86666666666666669627 0.86666666666666669627 0.050980392156862744391 1.0" />
             </material>
         </visual>
@@ -48,11 +50,11 @@
             <origin xyz="0 0 0" rpy="0 0 0" />
             <geometry>
-            <mesh filename="$(arg mesh_dir)fingertip_custom.stl"/>
+                <mesh filename="$(arg mesh_dir)fingertip_custom.stl" />
             </geometry>
         </collision>
         <inertial>
-            <origin xyz="0 0 0" rpy="0 0 0"/>
+            <origin xyz="0 0 0" rpy="0 0 0" />
             <mass value="0.0000000001" />
-            <inertia ixx="0.0000000001" ixy="0"  ixz="0" iyy="0.0000000001" iyz="0" izz="0.0000000001" />
+            <inertia ixx="0.0000000001" ixy="0" ixz="0" iyy="0.0000000001" iyz="0" izz="0.0000000001" />
         </inertial>
     </link>
@@ -61,8 +63,8 @@
             <origin xyz="0 0 0" rpy="0 0 0" />
             <geometry>
-            <mesh filename="$(arg mesh_dir)fingertip_custom.stl"/>
+                <mesh filename="$(arg mesh_dir)fingertip_custom.stl" />
             </geometry>
             <material name="fingertip_material">
-            <color rgba="0.86666666666666669627 0.86666666666666669627 0.050980392156862744391 1.0"/>
+                <color rgba="0.86666666666666669627 0.86666666666666669627 0.050980392156862744391 1.0" />
             </material>
         </visual>
@@ -70,11 +72,11 @@
             <origin xyz="0 0 0" rpy="0 0 0" />
             <geometry>
-            <mesh filename="$(arg mesh_dir)fingertip_custom.stl"/>
+                <mesh filename="$(arg mesh_dir)fingertip_custom.stl" />
             </geometry>
         </collision>
         <inertial>
-            <origin xyz="0 0 0" rpy="0 0 0"/>
+            <origin xyz="0 0 0" rpy="0 0 0" />
             <mass value="0.0000000001" />
-            <inertia ixx="0.0000000001" ixy="0"  ixz="0" iyy="0.0000000001" iyz="0" izz="0.0000000001" />
+            <inertia ixx="0.0000000001" ixy="0" ixz="0" iyy="0.0000000001" iyz="0" izz="0.0000000001" />
         </inertial>
     </link>
@@ -83,8 +85,8 @@
             <origin xyz="0 0 0 " rpy="0 0 0" />
             <geometry>
-            <mesh filename="$(arg mesh_dir)fingertip_custom.stl"/>
+                <mesh filename="$(arg mesh_dir)fingertip_custom.stl" />
             </geometry>
             <material name="fingertip_material">
-            <color rgba="0.86666666666666669627 0.86666666666666669627 0.050980392156862744391 1.0"/>
+                <color rgba="0.86666666666666669627 0.86666666666666669627 0.050980392156862744391 1.0" />
             </material>
         </visual>
@@ -92,64 +94,64 @@
             <origin xyz="0 0 0" rpy="0 0 0" />
             <geometry>
-            <mesh filename="$(arg mesh_dir)fingertip_custom.stl"/>
+                <mesh filename="$(arg mesh_dir)fingertip_custom.stl" />
             </geometry>
         </collision>
         <inertial>
-            <origin xyz="0 0 0" rpy="0 0 0"/>
+            <origin xyz="0 0 0" rpy="0 0 0" />
             <mass value="0.0000000001" />
-            <inertia ixx="0.0000000001" ixy="0"  ixz="0" iyy="0.0000000001" iyz="0" izz="0.0000000001" />
+            <inertia ixx="0.0000000001" ixy="0" ixz="0" iyy="0.0000000001" iyz="0" izz="0.0000000001" />
         </inertial>
     </link>
     <joint name="finger1_tipbase2tip" type="fixed">
         <origin xyz="0 -0.017 0.0145" rpy="0 ${pi/2} ${pi}" />
-        <parent link="fingertip"/>
-        <child link="fingertip_new"/>
+        <parent link="fingertip" />
+        <child link="fingertip_new" />
     </joint>
     <joint name="finger2_tipbase2tip" type="fixed">
         <origin xyz="0 -0.017 0.0145" rpy="0 ${pi/2} ${pi}" />
-        <parent link="fingertip_2"/>
-        <child link="fingertip_2_new"/>
+        <parent link="fingertip_2" />
+        <child link="fingertip_2_new" />
     </joint>
     <joint name="finger3_tipbase2tip" type="fixed">
         <origin xyz="0 -0.017 0.0145" rpy="0 ${pi/2} ${pi}" />
-        <parent link="fingertip_3"/>
-        <child link="fingertip_3_new"/>
+        <parent link="fingertip_3" />
+        <child link="fingertip_3_new" />
     </joint>
     <joint name="thumb_tipbase2tip" type="fixed">
         <origin xyz="0 -0.03 -0.0145" rpy="0 ${pi/2} ${pi}" />
-        <parent link="thumb_fingertip"/>
-        <child link="thumb_fingertip_new"/>
+        <parent link="thumb_fingertip" />
+        <child link="thumb_fingertip_new" />
     </joint>
     <!-- the links and joints for fingertip frames (point contact) -->
-	<link name="finger1_tip_center"/>
-	<link name="finger2_tip_center"/>
-	<link name="finger3_tip_center"/>
-	<link name="thumb_tip_center"/>
-	<joint name="finger1_tip2center" type="fixed">
-        <origin rpy="0 0 0" xyz="0 0.04 0"/>
-        <parent link="fingertip_new"/>
-        <child link="finger1_tip_center"/>
+    <link name="finger1_tip_center" />
+    <link name="finger2_tip_center" />
+    <link name="finger3_tip_center" />
+    <link name="thumb_tip_center" />
+    <joint name="finger1_tip2center" type="fixed">
+        <origin rpy="0 0 0" xyz="0 0.04 0" />
+        <parent link="fingertip_new" />
+        <child link="finger1_tip_center" />
     </joint>
     <joint name="finger2_tip2center" type="fixed">
-        <origin rpy="0 0 0" xyz="0 0.04 0"/>
-        <parent link="fingertip_2_new"/>
-        <child link="finger2_tip_center"/>
+        <origin rpy="0 0 0" xyz="0 0.04 0" />
+        <parent link="fingertip_2_new" />
+        <child link="finger2_tip_center" />
     </joint>
     <joint name="finger3_tip2center" type="fixed">
-        <origin rpy="0 0 0" xyz="0 0.04 0"/>
-        <parent link="fingertip_3_new"/>
-        <child link="finger3_tip_center"/>
+        <origin rpy="0 0 0" xyz="0 0.04 0" />
+        <parent link="fingertip_3_new" />
+        <child link="finger3_tip_center" />
     </joint>
     <joint name="thumb_tip2center" type="fixed">
-        <origin rpy="0 0 0" xyz="0 0.04 0"/>
-        <parent link="thumb_fingertip_new"/>
-        <child link="thumb_tip_center"/>
+        <origin rpy="0 0 0" xyz="0 0.04 0" />
+        <parent link="thumb_fingertip_new" />
+        <child link="thumb_tip_center" />
     </joint>
     <!-- the links and joints for world frame -->
-    <link name="world"/>
+    <link name="world" />
     <joint name="world2hand" type="fixed">
         <origin xyz="0 0 0" rpy="${pi} 0 0" />
-        <parent link="world"/>
-        <child link="palm_lower"/>
+        <parent link="world" />
+        <child link="palm_lower" />
     </joint>
 </robot>

File: my_robot_description/urdf/others/leaphand.urdf (robot description, URDF)
Before this commit: robot leap_hand, 26 links, 25 joints
Links:
- removed link dip
- removed link dip_2
- removed link dip_3
- removed link fingertip
- removed link fingertip_2
- removed link fingertip_2_new
- removed link fingertip_3
- removed link fingertip_3_new
- removed link fingertip_new
- removed link mcp_joint
- removed link mcp_joint_2
- removed link mcp_joint_3
- removed link pip
- removed link pip_2
- removed link pip_3
- removed link pip_4
- removed link thumb_dip
- removed link thumb_fingertip
- removed link thumb_fingertip_new
- removed link thumb_pip
- added link leap_link_0, mass 0.032; collision mesh filename=package://drake_models/leap_description/meshes/pip.stl; visual mesh filename=package://drake_models/leap_description/meshes/pip.stl
- added link leap_link_1, mass 0.044; collision mesh filename=package://drake_models/leap_description/meshes/mcp_joint.stl; visual mesh filename=package://drake_models/leap_description/meshes/mcp_joint.stl
- added link leap_link_10, mass 0.037; collision mesh filename=package://drake_models/leap_description/meshes/dip.stl; visual mesh filename=package://drake_models/leap_description/meshes/dip.stl
- added link leap_link_11, mass 0.016; collision mesh filename=package://drake_models/leap_description/meshes/fingertip_ba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; visual mesh filename=package://drake_models/leap_description/meshes/fingertip_ba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
- added link leap_link_12, mass 0.032; collision mesh filename=package://drake_models/leap_description/meshes/pip.stl; visual mesh filename=package://drake_models/leap_description/meshes/pip.stl
- added link leap_link_13, mass 0.003; collision mesh filename=package://drake_models/leap_description/meshes/thumb_pip.stl; visual mesh filename=package://drake_models/leap_description/meshes/thumb_pip.stl
- added link leap_link_14, mass 0.038; collision mesh filename=package://drake_models/leap_description/meshes/thumb_dip.stl; visual mesh filename=package://drake_models/leap_description/meshes/thumb_dip.stl
- added link leap_link_15, mass 0.049; collision mesh filename=package://drake_models/leap_description/meshes/thumb_finger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; visual mesh filename=package://drake_models/leap_description/meshes/thumb_finger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
- added link leap_link_16, mass 0.0000000001; collision mesh filename=package://drake_models/leap_description/meshes/fingertip_cu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; visual mesh filename=package://drake_models/leap_description/meshes/fingertip_cu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
- added link leap_link_17, mass 0.0000000001; collision mesh filename=package://drake_models/leap_description/meshes/fingertip_cu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; visual mesh filename=package://drake_models/leap_description/meshes/fingertip_cu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
- added link leap_link_18, mass 0.0000000001; collision mesh filename=package://drake_models/leap_description/meshes/fingertip_cu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; visual mesh filename=package://drake_models/leap_description/meshes/fingertip_cu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
- added link leap_link_19, mass 0.0000000001; collision mesh filename=package://drake_models/leap_description/meshes/fingertip_cu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; visual mesh filename=package://drake_models/leap_description/meshes/fingertip_cu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
- added link leap_link_2, mass 0.037; collision mesh filename=package://drake_models/leap_description/meshes/dip.stl; visual mesh filename=package://drake_models/leap_description/meshes/dip.stl
- added link leap_link_3, mass 0.016; collision mesh filename=package://drake_models/leap_description/meshes/fingertip_ba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; visual mesh filename=package://drake_models/leap_description/meshes/fingertip_ba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
- added link leap_link_4, mass 0.032; collision mesh filename=package://drake_models/leap_description/meshes/pip.stl; visual mesh filename=package://drake_models/leap_description/meshes/pip.stl
- added link leap_link_5, mass 0.044; collision mesh filename=package://drake_models/leap_description/meshes/mcp_joint.stl; visual mesh filename=package://drake_models/leap_description/meshes/mcp_joint.stl
- added link leap_link_6, mass 0.037; collision mesh filename=package://drake_models/leap_description/meshes/dip.stl; visual mesh filename=package://drake_models/leap_description/meshes/dip.stl
- added link leap_link_7, mass 0.016; collision mesh filename=package://drake_models/leap_description/meshes/fingertip_ba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; visual mesh filename=package://drake_models/leap_description/meshes/fingertip_ba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
- added link leap_link_8, mass 0.032; collision mesh filename=package://drake_models/leap_description/meshes/pip.stl; visual mesh filename=package://drake_models/leap_description/meshes/pip.stl
- added link leap_link_9, mass 0.044; collision mesh filename=package://drake_models/leap_description/meshes/mcp_joint.stl; visual mesh filename=package://drake_models/leap_description/meshes/mcp_joint.stl
- link palm_lower: geometry collision mesh filename=package://drake_models/leap_description/meshes/palm_lower.s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; visual box size=0.035 0.115 0.025
Joints:
- joint finger1_tip2center: parent fingertip_new -> leap_link_16
- joint finger1_tipbase2tip: child fingertip_new -> leap_link_16; parent fingertip -> leap_link_3
- joint finger2_tip2center: parent fingertip_2_new -> leap_link_17
- joint finger2_tipbase2tip: child fingertip_2_new -> leap_link_17; parent fingertip_2 -> leap_link_7
- joint finger3_tip2center: parent fingertip_3_new -> leap_link_18
- joint finger3_tipbase2tip: child fingertip_3_new -> leap_link_18; parent fingertip_3 -> leap_link_11
- joint joint_0: child pip -> leap_link_0; parent mcp_joint -> leap_link_1
- joint joint_1: child mcp_joint -> leap_link_1
- joint joint_10: child dip_3 -> leap_link_10; parent pip_3 -> leap_link_8
- joint joint_11: child fingertip_3 -> leap_link_11; parent dip_3 -> leap_link_10
- joint joint_12: child pip_4 -> leap_link_12
- joint joint_13: child thumb_pip -> leap_link_13; parent pip_4 -> leap_link_12
- joint joint_14: child thumb_dip -> leap_link_14; parent thumb_pip -> leap_link_13
- joint joint_15: child thumb_fingertip -> leap_link_15; parent thumb_dip -> leap_link_14
- joint joint_2: child dip -> leap_link_2; parent pip -> leap_link_0
- joint joint_3: child fingertip -> leap_link_3; parent dip -> leap_link_2
- joint joint_4: child pip_2 -> leap_link_4; parent mcp_joint_2 -> leap_link_5
- joint joint_5: child mcp_joint_2 -> leap_link_5
- joint joint_6: child dip_2 -> leap_link_6; parent pip_2 -> leap_link_4
- joint joint_7: child fingertip_2 -> leap_link_7; parent dip_2 -> leap_link_6
- joint joint_8: child pip_3 -> leap_link_8; parent mcp_joint_3 -> leap_link_9
- joint joint_9: child mcp_joint_3 -> leap_link_9
- joint thumb_tip2center: parent thumb_fingertip_new -> leap_link_19
- joint thumb_tipbase2tip: child thumb_fingertip_new -> leap_link_19; parent thumb_fingertip -> leap_link_15
